Commit message: fix: rotate lidar_joint 180° to match physical backward mounting

File: src/surveillance_bot_description/urdf/surveillance_bot.xacro (robot description, xacro)
@@ -173,5 +173,5 @@
 </joint>
 <joint name="lidar_joint" type="fixed">
-  <origin xyz="0.0875 0.0 0.155" rpy="0 0 0"/>
+  <origin xyz="0.0875 0.0 0.155" rpy="0 0 3.14159"/>
   <parent link="base_link"/>
   <child link="lidar_1"/>
